File: V1/dc-ac-8ch-v1.kicad_pcb (KiCad board)
At the start: 2 copper layers, 53 x 67.8 mm, 53 parts, among them J1 DB142V-5.08-4P, J2 DB142V-5.08-2P, J3 DB142V-5.08-4P, J4 DB142V-5.08-2P, U1 MOC3063S, U2 MOC3063S, U3 MOC3063S, U4 MOC3063S

Commit message: Update dc-ac-8ch-v1.kicad_pcb
Parts:
- moved REF** 11.0 mm to (156.5, 87.0)
Routing:
- net Net-(D9-G): track 20.2 -> 16.6 mm
- net Net-(D6-G): track 20.2 -> 16.6 mm
- net Net-(D12-G): track 20.2 -> 16.6 mm
- net Net-(D3-G): track 20.2 -> 16.6 mm
Changed lines of the file:
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@@
   )
   (footprint "Tales:Logo_Tramontina_25mm_Bottom" (layer "F.Cu")
-    (at 145.5 87.5)
+    (at 156.5 87)
     (descr "Tramontina Logo 25 mm")
     (attr through_hole)
@@
   (gr_rect (start 120 62.2) (end 173 130)
     (stroke (width 0.1) (type solid)) (fill none) (layer "Edge.Cuts"))
-  (gr_text "DC-AC-4CH-V1" (at 145.5 71.5) (layer "B.Cu")
+  (gr_text "DC-AC-4CH-V1" (at 133 87) (layer "B.Cu")
     (effects (font (size 1.5 1.3) (thickness 0.25) bold) (justify bottom mirror))
   )
-  (gr_text "INPUT 24VDC\nOUTPUT 220VAC 1A\n2023 TMASCHIO" (at 145.5 81) (layer "B.Cu")
+  (gr_text "INPUT 24VDC\nOUTPUT 220VAC 1A\n2023 TMASCHIO" (at 133 92) (layer "B.Cu")
     (effects (font (size 1 1) (thickness 0.15)) (justify bottom mirror))
   )
@@
   (segment (start 126 105.56) (end 124 107.56) (width 0.4) (layer "F.Cu") (net 14))
   (segment (start 126 105.5) (end 126 105.56) (width 0.4) (layer "F.Cu") (net 14))
-  (segment (start 124.92 94.08) (end 124.92 94.53) (width 0.6) (layer "F.Cu") (net 14))
-  (segment (start 126 93) (end 124.92 94.08) (width 0.6) (layer "F.Cu") (net 14))
   (segment (start 124 95.45) (end 124.92 94.53) (width 1) (layer "F.Cu") (net 14))
   (segment (start 124 97) (end 124 95.45) (width 1) (layer "F.Cu") (net 14))
-  (via (at 126 93) (size 0.8) (drill 0.4) (layers "F.Cu" "B.Cu") (net 14))
   (via (at 126 105.5) (size 0.6) (drill 0.3) (layers "F.Cu" "B.Cu") (net 14))
-  (segment (start 126 93) (end 126 105.5) (width 0.4) (layer "B.Cu") (net 14))
+  (via (at 124 95.45) (size 0.8) (drill 0.4) (layers "F.Cu" "B.Cu") (net 14))
+  (segment (start 124 95.45) (end 126 97.45) (width 0.4) (layer "B.Cu") (net 14))
+  (segment (start 126 97.45) (end 126 105.5) (width 0.4) (layer "B.Cu") (net 14))
   (segment (start 136.075 82.65) (end 136 82.575) (width 0.8) (layer "F.Cu") (net 15))
   (segment (start 138 82.65) (end 136.075 82.65) (width 0.8) (layer "F.Cu") (net 15))
@@
   (segment (start 138 105.5) (end 138 105.56) (width 0.4) (layer "F.Cu") (net 18))
   (segment (start 136 95.45) (end 136.92 94.53) (width 1) (layer "F.Cu") (net 18))
-  (segment (start 136.92 94.08) (end 136.92 94.53) (width 0.6) (layer "F.Cu") (net 18))
-  (segment (start 138 93) (end 136.92 94.08) (width 0.6) (layer "F.Cu") (net 18))
   (segment (start 138 105.56) (end 136 107.56) (width 0.4) (layer "F.Cu") (net 18))
   (via (at 138 105.5) (size 0.6) (drill 0.3) (layers "F.Cu" "B.Cu") (net 18))
-  (via (at 138 93) (size 0.8) (drill 0.4) (layers "F.Cu" "B.Cu") (net 18))
-  (segment (start 138 93) (end 138 105.5) (width 0.4) (layer "B.Cu") (net 18))
+  (via (at 136 95.45) (size 0.8) (drill 0.4) (layers "F.Cu" "B.Cu") (net 18))
+  (segment (start 138 97.45) (end 138 105.5) (width 0.4) (layer "B.Cu") (net 18))
+  (segment (start 136 95.45) (end 138 97.45) (width 0.4) (layer "B.Cu") (net 18))
   (segment (start 150 82.65) (end 148.075 82.65) (width 0.8) (layer "F.Cu") (net 19))
   (segment (start 148.075 82.65) (end 148 82.575) (width 0.8) (layer "F.Cu") (net 19))
@@
   (segment (start 150 105.56) (end 148 107.56) (width 0.4) (layer "F.Cu") (net 22))
   (segment (start 148 97) (end 148 95.45) (width 1) (layer "F.Cu") (net 22))
-  (segment (start 150 93) (end 148.92 94.08) (width 0.6) (layer "F.Cu") (net 22))
-  (segment (start 148.92 94.08) (end 148.92 94.53) (width 0.6) (layer "F.Cu") (net 22))
-  (via (at 150 93) (size 0.8) (drill 0.4) (layers "F.Cu" "B.Cu") (net 22))
   (via (at 150 105.5) (size 0.6) (drill 0.3) (layers "F.Cu" "B.Cu") (net 22))
-  (segment (start 150 93) (end 150 105.5) (width 0.4) (layer "B.Cu") (net 22))
+  (via (at 148 95.45) (size 0.8) (drill 0.4) (layers "F.Cu" "B.Cu") (net 22))
+  (segment (start 148 95.45) (end 150 97.45) (width 0.4) (layer "B.Cu") (net 22))
+  (segment (start 150 97.45) (end 150 105.5) (width 0.4) (layer "B.Cu") (net 22))
   (segment (start 160.075 82.65) (end 160 82.575) (width 0.8) (layer "F.Cu") (net 23))
   (segment (start 162 82.65) (end 160.075 82.65) (width 0.8) (layer "F.Cu") (net 23))
@@
   (segment (start 162 105.56) (end 160 107.56) (width 0.4) (layer "F.Cu") (net 26))
   (segment (start 162 105.5) (end 162 105.56) (width 0.4) (layer "F.Cu") (net 26))
-  (segment (start 160.92 94.08) (end 160.92 94.53) (width 0.6) (layer "F.Cu") (net 26))
-  (segment (start 162 93) (end 160.92 94.08) (width 0.6) (layer "F.Cu") (net 26))
   (segment (start 160 97) (end 160 95.45) (width 1) (layer "F.Cu") (net 26))
-  (via (at 162 93) (size 0.8) (drill 0.4) (layers "F.Cu" "B.Cu") (net 26))
+  (via (at 160 95.45) (size 0.8) (drill 0.4) (layers "F.Cu" "B.Cu") (net 26))
   (via (at 162 105.5) (size 0.6) (drill 0.3) (layers "F.Cu" "B.Cu") (net 26))
-  (segment (start 162 93) (end 162 105.5) (width 0.4) (layer "B.Cu") (net 26))
+  (segment (start 160 95.45) (end 162 97.45) (width 0.4) (layer "B.Cu") (net 26))
+  (segment (start 162 97.45) (end 162 105.5) (width 0.4) (layer "B.Cu") (net 26))
   (segment (start 164 82.825) (end 163.825 82.825) (width 0.6) (layer "F.Cu") (net 27))
   (segment (start 151 66.88) (end 151 74.5) (width 2) (layer "F.Cu") (net 27))
