File: V1/dc-ac-4ch-v1.kicad_pcb (KiCad board)
At the start: 2 copper layers, 53 x 67.8 mm, 53 parts, among them J1 DB142V-5.08-4P, J2 DB142V-5.08-2P, J3 DB142V-5.08-4P, J4 DB142V-5.08-2P, U1 MOC3063S, U2 MOC3063S, U3 MOC3063S, U4 MOC3063S

Commit message: Repo cleanup
Other:
- board text added: "SUPORTES PCI METALTEX SP7 1x pé macho 9 mm 1x pé fêmea 9 mm 1x espaçador 20 mm 3x espaçador 5mm Comprimento total 53 mm Largura da placa 67,8 mm"
- board text removed: "SUPORTES PCI METALTEX SP7 1x pé macho 9 mm 1x pé fêmea 9 mm 2x espaçadores 30 mm 1x espaçador 20 mm Comprimento total 98 mm Largura da placa 67,8 mm"
Changed lines of the file:
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@@
   (footprint "Tales:TerminalBlock_Dibo_DB142V-5.08-4P_1x04_P5.08mm_Vertical" (layer "F.Cu")
     (at 131 125.62)
+    (property "JLCPCB BOM" "1")
+    (property "LCSC Part #" "C2898701")
+    (property "Mfr" "DIBO")
+    (property "Mfr Part #" "DB142V-5.08-4P")
+    (property "Package" "01x04 P5.08")
     (property "Sheetfile" "dc-ac-4ch-v1.kicad_sch")
     (property "Sheetname" "")
+    (property "Technology" "Spring Cage")
+    (property "Vendor" "JLCPCB")
+    (property "Vendor Part #" "C2898701")
     (property "ki_description" "Generic connector, single row, 01x04, script generated (kicad-library-utils/schlib/autogen/connector/)")
     (property "ki_keywords" "connector")
@@
   (footprint "Tales:TerminalBlock_Dibo_DB142V-5.08-4P_1x04_P5.08mm_Vertical" (layer "F.Cu")
     (at 151 66.88 180)
+    (property "JLCPCB BOM" "1")
+    (property "LCSC Part #" "C2898701")
+    (property "Mfr" "DIBO")
+    (property "Mfr Part #" "DB142V-5.08-4P")
+    (property "Package" "01x04 P5.08")
     (property "Sheetfile" "dc-ac-4ch-v1.kicad_sch")
     (property "Sheetname" "")
+    (property "Technology" "Spring Cage")
+    (property "Vendor" "JLCPCB")
+    (property "Vendor Part #" "C2898701")
     (property "ki_description" "Generic connector, single row, 01x04, script generated (kicad-library-utils/schlib/autogen/connector/)")
     (property "ki_keywords" "connector")
@@
     (property "Mfr" "DIBO")
     (property "Mfr Part #" "DB142V-5.08-2P")
-    (property "Package" "01x08 P5.08")
+    (property "Package" "01x02 P5.08")
     (property "Sheetfile" "dc-ac-4ch-v1.kicad_sch")
     (property "Sheetname" "")
@@
     (property "Mfr" "DIBO")
     (property "Mfr Part #" "DB142V-5.08-2P")
-    (property "Package" "01x08 P5.08")
+    (property "Package" "01x02 P5.08")
     (property "Sheetfile" "dc-ac-4ch-v1.kicad_sch")
     (property "Sheetname" "")
@@
     (effects (font (size 1 1) (thickness 0.16) bold))
   )
-  (gr_text "SUPORTES PCI METALTEX SP7\n1x pé macho  9 mm\n1x pé fêmea 9 mm\n2x espaçadores 30 mm\n1x espaçador 20 mm\nComprimento total 98 mm\nLargura da placa 67,8 mm" (at 120.702 138.89) (layer "Cmts.User")
-    (effects (font (size 1.27 1.27) (thickness 0.0508)) (justify left))
+  (gr_text "SUPORTES PCI METALTEX SP7\n1x pé macho  9 mm\n1x pé fêmea 9 mm\n1x espaçador 20 mm\n3x espaçador 5mm\nComprimento total 53 mm\nLargura da placa 67,8 mm" (at 120 132) (layer "Cmts.User")
+    (effects (font (size 1 1) (thickness 0.15)) (justify left top))
   )
   (dimension (type aligned) (layer "Dwgs.User")
