File: V1/dc-ac-4ch-v1.kicad_sch (KiCad schematic)
At the start: 52 parts, among them J1 DB142V-5.08-4P, J2 DB142V-5.08-2P, J3 DB142V-5.08-4P, J4 DB142V-5.08-2P, U1 MOC3063S, U2 MOC3063S, U3 MOC3063S, U4 MOC3063S

Commit message: Repo cleanup
Parts:
- J1, J3: JLCPCB BOM (none) -> 1; LCSC Part # (none) -> C2898701; Mfr (none) -> DIBO; Mfr Part # (none) -> DB142V-5.08-4P; Package (none) -> 01x04 P5.08; Technology (none) -> Spring Cage; Vendor (none) -> JLCPCB; Vendor Part # (none) -> C2898701
- J2, J4: Package 01x08 P5.08 -> 01x02 P5.08
Changed lines of the file:
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@@
   )
   (symbol (lib_id "Connector_Generic:Conn_01x02") (at 256.54 160.02 0) (mirror x) (unit 1)
-    (in_bom yes) (on_board yes) (dnp no)
-    (property "Reference" "J4" (at 259.08 160.655 0)
-      (effects (font (size 1.27 1.27)) (justify left))
-    )
-    (property "Value" "DB142V-5.08-2P" (at 259.08 158.115 0)
-      (effects (font (size 1.27 1.27)) (justify left))
+    (in_bom yes) (on_board yes) (dnp no) (fields_autoplaced)
+    (property "Reference" "J4" (at 256.54 149.86 0)
+      (effects (font (size 1.27 1.27)))
+    )
+    (property "Value" "DB142V-5.08-2P" (at 256.54 152.4 0)
+      (effects (font (size 1.27 1.27)))
     )
     (property "Footprint" "Tales:TerminalBlock_Dibo_DB142V-5.08-2P_1x02_P5.08mm_Vertical" (at 256.54 160.02 0)
@@
       (effects (font (size 1.27 1.27)) hide)
     )
-    (property "LCSC Part #" "C2898699" (at 259.08 155.575 0)
-      (effects (font (size 1.27 1.27)) (justify left))
+    (property "LCSC Part #" "C2898699" (at 256.54 154.94 0)
+      (effects (font (size 1.27 1.27)))
     )
     (property "Mfr" "DIBO" (at 256.54 160.02 0)
@@
       (effects (font (size 1.27 1.27)) hide)
     )
-    (property "Package" "01x08 P5.08" (at 256.54 160.02 0)
+    (property "Package" "01x02 P5.08" (at 256.54 160.02 0)
       (effects (font (size 1.27 1.27)) hide)
     )
@@
   )
   (symbol (lib_id "Connector_Generic:Conn_01x04") (at 265.43 101.6 0) (unit 1)
-    (in_bom yes) (on_board yes) (dnp no)
-    (property "Reference" "J3" (at 264.16 110.49 0)
-      (effects (font (size 1.27 1.27)) (justify left))
-    )
-    (property "Value" "DB142V-5.08-4P" (at 264.16 113.03 0)
+    (in_bom yes) (on_board yes) (dnp no) (fields_autoplaced)
+    (property "Reference" "J3" (at 267.97 100.965 0)
+      (effects (font (size 1.27 1.27)) (justify left))
+    )
+    (property "Value" "DB142V-5.08-4P" (at 267.97 103.505 0)
       (effects (font (size 1.27 1.27)) (justify left))
     )
@@
     )
     (property "Datasheet" "~" (at 265.43 101.6 0)
+      (effects (font (size 1.27 1.27)) hide)
+    )
+    (property "JLCPCB BOM" "1" (at 265.43 101.6 0)
+      (effects (font (size 1.27 1.27)) hide)
+    )
+    (property "LCSC Part #" "C2898701" (at 267.97 106.045 0)
+      (effects (font (size 1.27 1.27)) (justify left))
+    )
+    (property "Mfr" "DIBO" (at 265.43 101.6 0)
+      (effects (font (size 1.27 1.27)) hide)
+    )
+    (property "Mfr Part #" "DB142V-5.08-4P" (at 265.43 101.6 0)
+      (effects (font (size 1.27 1.27)) hide)
+    )
+    (property "Vendor" "JLCPCB" (at 265.43 101.6 0)
+      (effects (font (size 1.27 1.27)) hide)
+    )
+    (property "Vendor Part #" "C2898701" (at 265.43 101.6 0)
+      (effects (font (size 1.27 1.27)) hide)
+    )
+    (property "Package" "01x04 P5.08" (at 265.43 101.6 0)
+      (effects (font (size 1.27 1.27)) hide)
+    )
+    (property "Technology" "Spring Cage" (at 265.43 101.6 0)
       (effects (font (size 1.27 1.27)) hide)
     )
@@
   )
   (symbol (lib_id "Connector_Generic:Conn_01x02") (at 34.29 170.18 0) (mirror y) (unit 1)
-    (in_bom yes) (on_board yes) (dnp no)
-    (property "Reference" "J2" (at 35.56 176.53 0)
-      (effects (font (size 1.27 1.27)) (justify left))
-    )
-    (property "Value" "DB142V-5.08-2P" (at 35.56 179.07 0)
+    (in_bom yes) (on_board yes) (dnp no) (fields_autoplaced)
+    (property "Reference" "J2" (at 31.75 169.545 0)
+      (effects (font (size 1.27 1.27)) (justify left))
+    )
+    (property "Value" "DB142V-5.08-2P" (at 31.75 172.085 0)
       (effects (font (size 1.27 1.27)) (justify left))
     )
@@
       (effects (font (size 1.27 1.27)) hide)
     )
-    (property "LCSC Part #" "C2898699" (at 35.56 181.61 0)
+    (property "LCSC Part #" "C2898699" (at 31.75 174.625 0)
       (effects (font (size 1.27 1.27)) (justify left))
     )
@@
       (effects (font (size 1.27 1.27)) hide)
     )
-    (property "Package" "01x08 P5.08" (at 34.29 170.18 0)
+    (property "Package" "01x02 P5.08" (at 34.29 170.18 0)
       (effects (font (size 1.27 1.27)) hide)
     )
@@
   (symbol (lib_id "Connector_Generic:Conn_01x04") (at 24.13 114.3 180) (unit 1)
     (in_bom yes) (on_board yes) (dnp no) (fields_autoplaced)
-    (property "Reference" "J1" (at 24.13 104.14 0)
+    (property "Reference" "J1" (at 24.13 101.6 0)
       (effects (font (size 1.27 1.27)))
     )
-    (property "Value" "DB142V-5.08-4P" (at 24.13 106.68 0)
+    (property "Value" "DB142V-5.08-4P" (at 24.13 104.14 0)
       (effects (font (size 1.27 1.27)))
     )
@@
       (effects (font (size 1.27 1.27)) hide)
     )
+    (property "JLCPCB BOM" "1" (at 24.13 114.3 0)
+      (effects (font (size 1.27 1.27)) hide)
+    )
+    (property "LCSC Part #" "C2898701" (at 24.13 106.68 0)
+      (effects (font (size 1.27 1.27)))
+    )
+    (property "Mfr" "DIBO" (at 24.13 114.3 0)
+      (effects (font (size 1.27 1.27)) hide)
+    )
+    (property "Mfr Part #" "DB142V-5.08-4P" (at 24.13 114.3 0)
+      (effects (font (size 1.27 1.27)) hide)
+    )
+    (property "Vendor" "JLCPCB" (at 24.13 114.3 0)
+      (effects (font (size 1.27 1.27)) hide)
+    )
+    (property "Vendor Part #" "C2898701" (at 24.13 114.3 0)
+      (effects (font (size 1.27 1.27)) hide)
+    )
+    (property "Package" "01x04 P5.08" (at 24.13 114.3 0)
+      (effects (font (size 1.27 1.27)) hide)
+    )
+    (property "Technology" "Spring Cage" (at 24.13 114.3 0)
+      (effects (font (size 1.27 1.27)) hide)
+    )
